Commit message: updates

File: urdf/turtlebot3_burger_custom.gazebo.xacro (robot description, xacro)
@@ -7,7 +7,7 @@
     <material>Gazebo/DarkGrey</material>
   </gazebo>
-  <gazebo reference="wheel_left_link">
-    <mu1>0.5</mu1>
-    <mu2>0.5</mu2>
+<gazebo reference="wheel_left_link">
+    <mu1>0.1</mu1>
+    <mu2>0.1</mu2>
     <kp>500000.0</kp>
     <kd>10.0</kd>
@@ -18,6 +18,6 @@
   </gazebo>
   <gazebo reference="wheel_right_link">
-    <mu1>0.5</mu1>
-    <mu2>0.5</mu2>
+    <mu1>0.1</mu1>
+    <mu2>0.1</mu2>
     <kp>500000.0</kp>
     <kd>10.0</kd>

File: urdf/turtlebot3_burger_custom.urdf.xacro (robot description, xacro)
@@ -31,8 +31,8 @@
     </inertial>
   </link>
-  <joint name="wheel_left_joint" type="continuous">
+    <joint name="wheel_left_joint" type="continuous">
     <parent link="base_link"/>
     <child link="wheel_left_link"/>
-    <origin xyz="0.0 0.08 -0.013" rpy="-1.57 0 0"/>
+    <origin xyz="0.0 0.08 0.023" rpy="-1.57 0 0"/>
     <axis xyz="0 0 1"/>
   </joint>
@@ -62,5 +62,5 @@
     <parent link="base_link"/>
     <child link="wheel_right_link"/>
-    <origin xyz="0.0 -0.080 -0.013" rpy="-1.57 0 0"/>
+    <origin xyz="0.0 -0.080 0.023" rpy="-1.57 0 0"/>
     <axis xyz="0 0 1"/>
   </joint>
@@ -94,15 +94,9 @@
   <link name="caster_back_link">
     <collision>
-      <origin xyz="0 0.018 0" rpy="0 0 0"/>
+      <origin xyz="0 0.001 0" rpy="0 0 0"/>
       <geometry>
-        <box size="0.030 0.044 0.020"/>
+        <box size="0.030 0.009 0.020"/>
       </geometry>
     </collision>
-    <visual>
-         <origin xyz="0 0.018 0" rpy="0 0 0"/>
-      <geometry>
-        <box size="0.030 0.044 0.020"/>
-      </geometry>
-    </visual>
     <inertial>
       <origin xyz="0 0 0" />

Commit message: change mesh resources

File: urdf/turtlebot3_burger_custom.gazebo.xacro (robot description, xacro)
@@ -42,4 +42,9 @@
     </sensor>
     <material>Gazebo/FlatBlack</material>
+  </gazebo>
+ <gazebo reference="camera_link">
+    <material>
+      <mesh filename="package://ballast_sim/meshes/sensors/D435i.stl" scale="0.001 0.001 0.001"/>
+    </material>
   </gazebo>
   <gazebo>

Commit message: change mesh resources

File: urdf/turtlebot3_burger_custom.gazebo.xacro (robot description, xacro)
@@ -44,7 +44,9 @@
   </gazebo>
  <gazebo reference="camera_link">
-    <material>
-      <mesh filename="package://ballast_sim/meshes/sensors/D435i.stl" scale="0.001 0.001 0.001"/>
-    </material>
+    <visual>
+	<geometry>
+          <mesh filename="package://ballast_sim/meshes/sensors/D435i.stl" scale="0.001 0.001 0.001"/>
+    	<geometry>
+</visual>
   </gazebo>
   <gazebo>

Commit message: change mesh resources

File: urdf/turtlebot3_burger_custom.gazebo.xacro (robot description, xacro)
@@ -47,5 +47,5 @@
 	<geometry>
           <mesh filename="package://ballast_sim/meshes/sensors/D435i.stl" scale="0.001 0.001 0.001"/>
-    	<geometry>
+    	</geometry>
 </visual>
   </gazebo>

Commit message: change mesh resources

File: urdf/turtlebot3_burger_custom.gazebo.xacro (robot description, xacro)
@@ -44,9 +44,4 @@
   </gazebo>
  <gazebo reference="camera_link">
-    <visual>
-	<geometry>
-          <mesh filename="package://ballast_sim/meshes/sensors/D435i.stl" scale="0.001 0.001 0.001"/>
-    	</geometry>
-</visual>
   </gazebo>
   <gazebo>

Commit message: rotate tag

File: urdf/turtlebot3_burger_custom.gazebo.xacro (robot description, xacro)
@@ -5,5 +5,5 @@
   <xacro:arg name="camera_visual" default="true"/>
   <gazebo reference="base_link">
-    <material>Gazebo/DarkGrey</material>
+    <material>Gazebo/Purple</material>
   </gazebo>
 <gazebo reference="wheel_left_link">
