Commit message: new topic name

File: urdf/turtlebot3_burger_custom.urdf.xacro (robot description, xacro)
@@ -172,16 +172,16 @@
     </collision>
   </link>
-  <joint name="camera_rgb_joint" type="fixed">
+  <joint name="camera_color_joint" type="fixed">
     <origin xyz="0.003 0.011 0.009" rpy="0 0 0"/>
     <parent link="camera_link"/>
-    <child link="camera_rgb_frame"/>
-  </joint>
-  <link name="camera_rgb_frame"/>
-  <joint name="camera_rgb_optical_joint" type="fixed">
+    <child link="camera_color_frame"/>
+  </joint>
+  <link name="camera_color_frame"/>
+  <joint name="camera_color_optical_joint" type="fixed">
     <origin xyz="0 0 0" rpy="-1.57 0 -1.57"/>
-    <parent link="camera_rgb_frame"/>
-    <child link="camera_rgb_optical_frame"/>
-  </joint>
-  <link name="camera_rgb_optical_frame"/>
+    <parent link="camera_color_frame"/>
+    <child link="camera_color_optical_frame"/>
+  </joint>
+  <link name="camera_color_optical_frame"/>
    <joint name="flashlight_joint" type="fixed">
 	<origin xyz="0.073 -0.011 0.2" rpy="0 0.3 0"/>

Commit message: change mesh resources

File: urdf/turtlebot3_burger_custom.urdf.xacro (robot description, xacro)
@@ -13,5 +13,5 @@
       <origin xyz="-0.032 0 0.0" rpy="0 0 0"/>
       <geometry>
-        <mesh filename="package://turtlebot3_description/meshes/bases/burger_base.stl" scale="0.001 0.001 0.001"/>
+        <mesh filename="package://ballast_sim/meshes/bases/burger_base.stl" scale="0.001 0.001 0.001"/>
       </geometry>
       <material name="light_black"/>
@@ -41,5 +41,5 @@
       <origin xyz="0 0 0" rpy="1.57 0 0"/>
       <geometry>
-        <mesh filename="package://turtlebot3_description/meshes/wheels/left_tire.stl" scale="0.001 0.001 0.001"/>
+        <mesh filename="package://ballast_sim/meshes/wheels/left_tire.stl" scale="0.001 0.001 0.001"/>
       </geometry>
       <material name="dark"/>
@@ -75,5 +75,5 @@
       <origin xyz="0 0 0" rpy="1.57 0 0"/>
       <geometry>
-        <mesh filename="package://turtlebot3_description/meshes/wheels/right_tire.stl" scale="0.001 0.001 0.001"/>
+        <mesh filename="package://ballast_sim/meshes/wheels/right_tire.stl" scale="0.001 0.001 0.001"/>
       </geometry>
       <material name="dark"/>
@@ -140,5 +140,5 @@
       <origin xyz="0 0 0.0" rpy="0 0 0"/>
       <geometry>
-        <mesh filename="package://turtlebot3_description/meshes/sensors/lds.stl" scale="0.001 0.001 0.001"/>
+        <mesh filename="package://ballast_sim/meshes/sensors/lds.stl" scale="0.001 0.001 0.001"/>
       </geometry>
       <material name="dark"/>

Commit message: change mesh resources

File: urdf/turtlebot3_burger_custom.urdf.xacro (robot description, xacro)
@@ -168,5 +168,5 @@
       <origin xyz="0.005 0.0 0.013" rpy="0 0 0"/>
       <geometry>
-        <box size="0.015 0.030 0.027"/>
+                <mesh filename="package://ballast_sim/meshes/sensors/D435i.stl" scale="0.001 0.001 0.001"/>
       </geometry>
     </collision>

Commit message: change mesh resources

File: urdf/turtlebot3_burger_custom.urdf.xacro (robot description, xacro)
@@ -160,5 +160,5 @@
  <joint name="camera_joint" type="fixed">
 <!--	<origin xyz="0.073 -0.011 0.084" rpy="0 0.349 0"/> -->
-<origin xyz="0.073 -0.011 0.2" rpy="0 0.157 0"/>
+<origin xyz="0.073 -0.011 0.2" rpy="0 0 0"/>
     <parent link="base_link"/>
     <child link="camera_link"/>

Commit message: change mesh resources

File: urdf/turtlebot3_burger_custom.urdf.xacro (robot description, xacro)
@@ -168,5 +168,5 @@
       <origin xyz="0.005 0.0 0.013" rpy="0 0 0"/>
       <geometry>
-                <mesh filename="package://ballast_sim/meshes/sensors/D435i.stl" scale="0.001 0.001 0.001"/>
+         <mesh filename="package://ballast_sim/meshes/sensors/D435i.stl" scale="0.001 0.001 0.001"/>
       </geometry>
     </collision>

Commit message: change mesh resources

File: urdf/turtlebot3_burger_custom.urdf.xacro (robot description, xacro)
@@ -165,10 +165,10 @@
   </joint>
   <link name="camera_link">
-    <collision>
+    <visual>
       <origin xyz="0.005 0.0 0.013" rpy="0 0 0"/>
       <geometry>
          <mesh filename="package://ballast_sim/meshes/sensors/D435i.stl" scale="0.001 0.001 0.001"/>
       </geometry>
-    </collision>
+    </visual>
   </link>
   <joint name="camera_color_joint" type="fixed">

Commit message: change mesh resources

File: urdf/turtlebot3_burger_custom.urdf.xacro (robot description, xacro)
@@ -170,4 +170,5 @@
          <mesh filename="package://ballast_sim/meshes/sensors/D435i.stl" scale="0.001 0.001 0.001"/>
       </geometry>
+      <material name="light_black"/>
     </visual>
   </link>

Commit message: change mesh resources

File: urdf/turtlebot3_burger_custom.urdf.xacro (robot description, xacro)
@@ -136,4 +136,5 @@
     <origin xyz="-0.032 0 0.172" rpy="0 0 0"/>
   </joint>
+<!--
   <link name="base_scan">
     <visual>
@@ -158,4 +159,5 @@
     </inertial>
   </link>
+  -->
  <joint name="camera_joint" type="fixed">
 <!--	<origin xyz="0.073 -0.011 0.084" rpy="0 0.349 0"/> -->
@@ -202,5 +204,5 @@
         <box size="0.015 0.030 0.027"/>
       </geometry>
-      <material name="dark"/>
+      <material name="light_black"/>
     </visual>
   </link>

Commit message: change mesh resources

File: urdf/turtlebot3_burger_custom.urdf.xacro (robot description, xacro)
@@ -131,4 +131,5 @@
   </joint>
   <link name="imu_link"/>
+<!--
   <joint name="scan_joint" type="fixed">
     <parent link="base_link"/>
@@ -136,7 +137,6 @@
     <origin xyz="-0.032 0 0.172" rpy="0 0 0"/>
   </joint>
-<!--
   <link name="base_scan">
-    <visual>
+   <visual>
       <origin xyz="0 0 0.0" rpy="0 0 0"/>
       <geometry>

Commit message: change mesh resources

File: urdf/turtlebot3_burger_custom.urdf.xacro (robot description, xacro)
@@ -170,5 +170,5 @@
       <origin xyz="0.005 0.0 0.013" rpy="0 0 0"/>
       <geometry>
-         <mesh filename="package://ballast_sim/meshes/sensors/D435i.stl" scale="0.001 0.001 0.001"/>
+         <mesh filename="package://ballast_sim/meshes/sensors/D435i.stl" scale="1 1 1"/>
       </geometry>
       <material name="light_black"/>

Commit message: change mesh resources

File: urdf/turtlebot3_burger_custom.urdf.xacro (robot description, xacro)
@@ -170,5 +170,5 @@
       <origin xyz="0.005 0.0 0.013" rpy="0 0 0"/>
       <geometry>
-         <mesh filename="package://ballast_sim/meshes/sensors/D435i.stl" scale="1 1 1"/>
+         <mesh filename="package://ballast_sim/meshes/sensors/d435.dae" scale="1 1 1"/>
       </geometry>
       <material name="light_black"/>

Commit message: change mesh resources

File: urdf/turtlebot3_burger_custom.urdf.xacro (robot description, xacro)
@@ -170,5 +170,5 @@
       <origin xyz="0.005 0.0 0.013" rpy="0 0 0"/>
       <geometry>
-         <mesh filename="package://ballast_sim/meshes/sensors/d435.dae" scale="1 1 1"/>
+         <mesh filename="package://ballast_sim/meshes/sensors/D435i.stl" scale="1 1 1"/>
       </geometry>
       <material name="light_black"/>

Commit message: change mesh resources

File: urdf/turtlebot3_burger_custom.urdf.xacro (robot description, xacro)
@@ -199,5 +199,5 @@
       </geometry>
     </collision>
-       <visual>
+     <!--  <visual>
       <origin xyz="0 0 0.0" rpy="0 0 0"/>
       <geometry>
@@ -205,5 +205,5 @@
       </geometry>
       <material name="light_black"/>
-    </visual>
+    </visual> -->
   </link>
 </robot>

Commit message: update

File: urdf/turtlebot3_burger_custom.urdf.xacro (robot description, xacro)
@@ -162,5 +162,5 @@
  <joint name="camera_joint" type="fixed">
 <!--	<origin xyz="0.073 -0.011 0.084" rpy="0 0.349 0"/> -->
-<origin xyz="0.073 -0.011 0.2" rpy="0 0 0"/>
+<origin xyz="0.01 -0.011 0.16" rpy="0 0 0"/>
     <parent link="base_link"/>
     <child link="camera_link"/>

Commit message: update

File: urdf/turtlebot3_burger_custom.urdf.xacro (robot description, xacro)
@@ -162,5 +162,5 @@
  <joint name="camera_joint" type="fixed">
 <!--	<origin xyz="0.073 -0.011 0.084" rpy="0 0.349 0"/> -->
-<origin xyz="0.01 -0.011 0.16" rpy="0 0 0"/>
+<origin xyz="0.01 0.032 0.16" rpy="0 0 0"/>
     <parent link="base_link"/>
     <child link="camera_link"/>
@@ -168,5 +168,5 @@
   <link name="camera_link">
     <visual>
-      <origin xyz="0.005 0.0 0.013" rpy="0 0 0"/>
+      <origin xyz="0.0 0.0 0.0" rpy="0 0 0"/>
       <geometry>
          <mesh filename="package://ballast_sim/meshes/sensors/D435i.stl" scale="1 1 1"/>
@@ -176,5 +176,5 @@
   </link>
   <joint name="camera_color_joint" type="fixed">
-    <origin xyz="0.003 0.011 0.009" rpy="0 0 0"/>
+    <origin xyz="0.0 -0.032 0.0" rpy="0 0 0"/>
     <parent link="camera_link"/>
     <child link="camera_color_frame"/>
